File: Placa_Miguel_Angel/eProject/Placa_1.brd (EAGLE design)
At the start: 100 x 100 mm, 20 parts, among them Q1 IRF510, Q2 2N2907A

Commit message: se termino la placa a soldar
Parts:
- removed Q1: IRF510, transistor-fet:TO220
- added Q3: IRF530, transistor-power:TO220BV
- moved OUT 153.9 mm to (87.6, 65.2), turned to 270 degrees
- moved L2 127.4 mm to (59.9, 81.1)
- moved SR540 126.8 mm to (85.1, 79.6), turned to 180 degrees
- moved R4 119.6 mm to (80.3, 21.7), turned to 180 degrees
- moved R2 115.0 mm to (66.4, 22.4)
- moved R3 111.0 mm to (80.6, 14.7), turned to 180 degrees
- moved C3 105.9 mm to (45.6, 81.5)
- moved R1 105.8 mm to (66.3, 14.4)
- moved MCP6002 104.8 mm to (74.1, 37.7)
- moved L1 97.4 mm to (30.2, 81.5)
- moved C2 93.5 mm to (70.8, 64.5), turned to 270 degrees
- moved R5 90.7 mm to (46.2, 59.8), turned to 180 degrees
- moved Q2 85.1 mm to (35.1, 42.2), turned to 180 degrees
- moved PRESET 82.6 mm to (39.8, 12.0)
- moved C1 80.8 mm to (20.0, 65.7), turned to 270 degrees
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Connections:
- net GND: now also Q3.S; no longer Q1.3
- net N$2: now also Q3.D; no longer Q1.2
- net N$9: now also Q3.G; no longer Q1.1
Routing:
- net VCC: track 0.00 -> 195.5 mm
- net GND: track 0.00 -> 112.7 mm
- net VOUT: track 0.00 -> 94.0 mm
- net N$8: track 0.00 -> 58.4 mm
- net N$6: track 0.00 -> 45.2 mm
- net N$1: track 0.00 -> 41.9 mm
- net N$2: track 0.00 -> 40.2 mm
- net N$3: track 0.00 -> 32.9 mm
- net N$4: track 0.00 -> 25.6 mm
- net N$7: track 0.00 -> 20.3 mm
- net N$5: track 0.00 -> 19.6 mm
- net N$9: track 0.00 -> 5.35 mm
- added copper zone on layer 16, net GND
Other:
- board size 100 x 100 mm -> 100 x 100.2 mm
