File: Placa_Miguel_Angel/eProject/Placa_1.sch (EAGLE design)
At the start: 20 parts, among them Q1 IRF510, Q2 2N2907A

Commit message: se termino la placa a soldar
Parts:
- removed Q1: IRF510, transistor-fet:IRF510
- added Q3: IRF530, transistor-power:IRF530
Connections:
- net GND: now also Q3.S; no longer Q1.S
- net N$2: now also Q3.D; no longer Q1.D
- net N$9: now also Q3.G; no longer Q1.G
Changed lines of the file:
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@@
 <part name="L2" library="con-ptr500" library_urn="urn:adsk.eagle:library:181" deviceset="AK550/2" device="" package3d_urn="urn:adsk.eagle:package:9907/1"/>
 <part name="C3" library="rcl" library_urn="urn:adsk.eagle:library:334" deviceset="C-EU" device="075-052X106" package3d_urn="urn:adsk.eagle:package:23650/1" value="4.7u"/>
-<part name="Q1" library="transistor-fet" library_urn="urn:adsk.eagle:library:396" deviceset="IRF510" device="" package3d_urn="urn:adsk.eagle:package:28520/1"/>
 <part name="SUPPLY1" library="supply2" library_urn="urn:adsk.eagle:library:372" deviceset="GND" device=""/>
 <part name="SR540" library="diode" library_urn="urn:adsk.eagle:library:210" deviceset="DIODE-" device="DO27-15" package3d_urn="urn:adsk.eagle:package:43337/1"/>
@@
 <part name="Q2" library="transistor-pnp" library_urn="urn:adsk.eagle:library:399" deviceset="2N2907*" device="" package3d_urn="urn:adsk.eagle:package:29207/1" technology="A"/>
 <part name="R5" library="rcl" library_urn="urn:adsk.eagle:library:334" deviceset="R-EU_" device="0207/10" package3d_urn="urn:adsk.eagle:package:23491/1"/>
+<part name="Q3" library="transistor-power" library_urn="urn:adsk.eagle:library:400" deviceset="IRF530" device="" package3d_urn="urn:adsk.eagle:package:29484/3"/>
 </parts>
 <sheets>
@@
 <instance part="L2" gate="-2" x="149.86" y="50.8" rot="MR0"/>
 <instance part="C3" gate="G$1" x="139.7" y="60.96" rot="R90"/>
-<instance part="Q1" gate="G$1" x="127" y="48.26"/>
 <instance part="SUPPLY1" gate="GND" x="139.7" y="22.86"/>
 <instance part="SR540" gate="G$1" x="152.4" y="60.96"/>
@@
 <instance part="Q2" gate="G$1" x="96.52" y="38.1"/>
 <instance part="R5" gate="G$1" x="109.22" y="45.72" rot="R180"/>
+<instance part="Q3" gate="G$1" x="127" y="48.26"/>
 </instances>
 <busses>
@@
 <wire x1="127" y1="63.5" x2="127" y2="60.96" width="0.1524" layer="91"/>
 <pinref part="C3" gate="G$1" pin="1"/>
-<wire x1="127" y1="60.96" x2="132.08" y2="60.96" width="0.1524" layer="91"/>
-<pinref part="Q1" gate="G$1" pin="D"/>
-<wire x1="132.08" y1="60.96" x2="137.16" y2="60.96" width="0.1524" layer="91"/>
-<wire x1="132.08" y1="50.8" x2="132.08" y2="60.96" width="0.1524" layer="91"/>
-<junction x="132.08" y="60.96"/>
+<wire x1="127" y1="60.96" x2="129.54" y2="60.96" width="0.1524" layer="91"/>
+<pinref part="Q3" gate="G$1" pin="D"/>
+<wire x1="129.54" y1="60.96" x2="137.16" y2="60.96" width="0.1524" layer="91"/>
+<wire x1="129.54" y1="60.96" x2="129.54" y2="53.34" width="0.1524" layer="91"/>
+<junction x="129.54" y="60.96"/>
 </segment>
 </net>
@@
 <pinref part="SUPPLY1" gate="GND" pin="GND"/>
 <wire x1="144.78" y1="25.4" x2="139.7" y2="25.4" width="0.1524" layer="91"/>
-<wire x1="139.7" y1="25.4" x2="132.08" y2="25.4" width="0.1524" layer="91"/>
-<pinref part="Q1" gate="G$1" pin="S"/>
-<wire x1="132.08" y1="25.4" x2="132.08" y2="45.72" width="0.1524" layer="91"/>
 <pinref part="C2" gate="G$1" pin="-"/>
 <wire x1="162.56" y1="48.26" x2="162.56" y2="25.4" width="0.1524" layer="91"/>
@@
 <wire x1="68.58" y1="48.26" x2="68.58" y2="25.4" width="0.1524" layer="91"/>
 <wire x1="68.58" y1="25.4" x2="99.06" y2="25.4" width="0.1524" layer="91"/>
-<wire x1="99.06" y1="25.4" x2="132.08" y2="25.4" width="0.1524" layer="91"/>
+<wire x1="99.06" y1="25.4" x2="129.54" y2="25.4" width="0.1524" layer="91"/>
+<wire x1="129.54" y1="25.4" x2="139.7" y2="25.4" width="0.1524" layer="91"/>
 <wire x1="68.58" y1="25.4" x2="43.18" y2="25.4" width="0.1524" layer="91"/>
 <pinref part="VCC" gate="-2" pin="KL"/>
@@
 <junction x="99.06" y="25.4"/>
 <junction x="68.58" y="25.4"/>
-<junction x="132.08" y="25.4"/>
 <junction x="144.78" y="25.4"/>
 <junction x="162.56" y="25.4"/>
 <junction x="182.88" y="25.4"/>
+<pinref part="Q3" gate="G$1" pin="S"/>
+<wire x1="129.54" y1="43.18" x2="129.54" y2="25.4" width="0.1524" layer="91"/>
+<junction x="129.54" y="25.4"/>
 </segment>
 <segment>
@@
 <segment>
 <pinref part="R5" gate="G$1" pin="1"/>
-<pinref part="Q1" gate="G$1" pin="G"/>
-<wire x1="114.3" y1="45.72" x2="121.92" y2="45.72" width="0.1524" layer="91"/>
-</segment>
-</net>
+<wire x1="114.3" y1="45.72" x2="124.46" y2="45.72" width="0.1524" layer="91"/>
+<pinref part="Q3" gate="G$1" pin="G"/>
+</segment>
+</net>
